File: Diseños pcb/Proyecto semaforo/emisor/emisor.kicad_pcb (KiCad board)
At the start: 2 copper layers, 12 parts, among them J1 Input, J2 Output

Commit message: PCB de emisor, receptor y relays
Parts:
- added J1: Input, Connector_JST:JST_EH_B2B-EH-A_1x02_P2.50mm_Vertical, F.Cu at (178.2, 82.6)
- added J1: Input, Connector_JST:JST_EH_B2B-EH-A_1x02_P2.50mm_Vertical, F.Cu at (177.2, 17.5)
- added J1: Input, Connector_JST:JST_EH_B2B-EH-A_1x02_P2.50mm_Vertical, F.Cu at (202.6, 17.0)
- added J1: Input, Connector_JST:JST_EH_B2B-EH-A_1x02_P2.50mm_Vertical, F.Cu at (226.4, 16.6)
- added J1: Input, Connector_JST:JST_EH_B2B-EH-A_1x02_P2.50mm_Vertical, F.Cu at (94.1, 83.6)
- added J1: Input, Connector_JST:JST_EH_B2B-EH-A_1x02_P2.50mm_Vertical, F.Cu at (119.6, 83.0)
- added J1: Input, Connector_JST:JST_EH_B2B-EH-A_1x02_P2.50mm_Vertical, F.Cu at (143.3, 82.6)
- added J1: Input, Connector_JST:JST_EH_B2B-EH-A_1x02_P2.50mm_Vertical, F.Cu at (95.9, 62.7)
- added J1: Input, Connector_JST:JST_EH_B2B-EH-A_1x02_P2.50mm_Vertical, F.Cu at (121.3, 62.2)
- added J1: Input, Connector_JST:JST_EH_B2B-EH-A_1x02_P2.50mm_Vertical, F.Cu at (145.1, 61.8)
- added J1: Input, Connector_JST:JST_EH_B2B-EH-A_1x02_P2.50mm_Vertical, F.Cu at (95.6, 40.6)
- added J1: Input, Connector_JST:JST_EH_B2B-EH-A_1x02_P2.50mm_Vertical, F.Cu at (203.6, 82.0)
- added J1: Input, Connector_JST:JST_EH_B2B-EH-A_1x02_P2.50mm_Vertical, F.Cu at (121.1, 40.1)
- added J1: Input, Connector_JST:JST_EH_B2B-EH-A_1x02_P2.50mm_Vertical, F.Cu at (144.8, 39.7)
- added J1: Input, Connector_JST:JST_EH_B2B-EH-A_1x02_P2.50mm_Vertical, F.Cu at (96.9, 20.3)
- added J1: Input, Connector_JST:JST_EH_B2B-EH-A_1x02_P2.50mm_Vertical, F.Cu at (122.4, 19.8)
- added J1: Input, Connector_JST:JST_EH_B2B-EH-A_1x02_P2.50mm_Vertical, F.Cu at (146.1, 19.4)
- added J1: Input, Connector_JST:JST_EH_B2B-EH-A_1x02_P2.50mm_Vertical, F.Cu at (14.9, 85.6)
- added J1: Input, Connector_JST:JST_EH_B2B-EH-A_1x02_P2.50mm_Vertical, F.Cu at (40.3, 85.1)
- added J1: Input, Connector_JST:JST_EH_B2B-EH-A_1x02_P2.50mm_Vertical, F.Cu at (64.1, 84.6)
- added J1: Input, Connector_JST:JST_EH_B2B-EH-A_1x02_P2.50mm_Vertical, F.Cu at (15.4, 63.5)
- added J1: Input, Connector_JST:JST_EH_B2B-EH-A_1x02_P2.50mm_Vertical, F.Cu at (40.8, 63.0)
- added J1: Input, Connector_JST:JST_EH_B2B-EH-A_1x02_P2.50mm_Vertical, F.Cu at (227.4, 81.6)
- added J1: Input, Connector_JST:JST_EH_B2B-EH-A_1x02_P2.50mm_Vertical, F.Cu at (64.6, 62.5)
- added J1: Input, Connector_JST:JST_EH_B2B-EH-A_1x02_P2.50mm_Vertical, F.Cu at (16.6, 42.2)
- added J1: Input, Connector_JST:JST_EH_B2B-EH-A_1x02_P2.50mm_Vertical, F.Cu at (42.1, 41.6)
- added J1: Input, Connector_JST:JST_EH_B2B-EH-A_1x02_P2.50mm_Vertical, F.Cu at (65.8, 41.2)
- added J1: Input, Connector_JST:JST_EH_B2B-EH-A_1x02_P2.50mm_Vertical, F.Cu at (177.2, 62.0)
- added J1: Input, Connector_JST:JST_EH_B2B-EH-A_1x02_P2.50mm_Vertical, F.Cu at (202.6, 61.5)
- added J1: Input, Connector_JST:JST_EH_B2B-EH-A_1x02_P2.50mm_Vertical, F.Cu at (226.4, 61.0)
- added J1: Input, Connector_JST:JST_EH_B2B-EH-A_1x02_P2.50mm_Vertical, F.Cu at (177.2, 40.4)
- added J1: Input, Connector_JST:JST_EH_B2B-EH-A_1x02_P2.50mm_Vertical, F.Cu at (202.6, 39.9)
- added J1: Input, Connector_JST:JST_EH_B2B-EH-A_1x02_P2.50mm_Vertical, F.Cu at (226.4, 39.4)
- added J2: Output, Connector_JST:JST_EH_B2B-EH-A_1x02_P2.50mm_Vertical, F.Cu at (220.7, 84.0)
- added J2: Output, Connector_JST:JST_EH_B2B-EH-A_1x02_P2.50mm_Vertical, F.Cu at (219.7, 19.0)
- added J2: Output, Connector_JST:JST_EH_B2B-EH-A_1x02_P2.50mm_Vertical, F.Cu at (243.4, 18.5)
- added J2: Output, Connector_JST:JST_EH_B2B-EH-A_1x02_P2.50mm_Vertical, F.Cu at (194.2, 19.5)
- added J2: Output, Connector_JST:JST_EH_B2B-EH-A_1x02_P2.50mm_Vertical, F.Cu at (136.7, 85.0)
- added J2: Output, Connector_JST:JST_EH_B2B-EH-A_1x02_P2.50mm_Vertical, F.Cu at (160.4, 84.6)
- added J2: Output, Connector_JST:JST_EH_B2B-EH-A_1x02_P2.50mm_Vertical, F.Cu at (111.2, 85.5)
- added J2: Output, Connector_JST:JST_EH_B2B-EH-A_1x02_P2.50mm_Vertical, F.Cu at (138.4, 64.2)
- added J2: Output, Connector_JST:JST_EH_B2B-EH-A_1x02_P2.50mm_Vertical, F.Cu at (162.2, 63.7)
- added J2: Output, Connector_JST:JST_EH_B2B-EH-A_1x02_P2.50mm_Vertical, F.Cu at (113.0, 64.7)
- added J2: Output, Connector_JST:JST_EH_B2B-EH-A_1x02_P2.50mm_Vertical, F.Cu at (138.2, 42.1)
- added J2: Output, Connector_JST:JST_EH_B2B-EH-A_1x02_P2.50mm_Vertical, F.Cu at (244.5, 83.5)
- added J2: Output, Connector_JST:JST_EH_B2B-EH-A_1x02_P2.50mm_Vertical, F.Cu at (161.9, 41.6)
- added J2: Output, Connector_JST:JST_EH_B2B-EH-A_1x02_P2.50mm_Vertical, F.Cu at (112.7, 42.6)
- added J2: Output, Connector_JST:JST_EH_B2B-EH-A_1x02_P2.50mm_Vertical, F.Cu at (139.4, 21.8)
- added J2: Output, Connector_JST:JST_EH_B2B-EH-A_1x02_P2.50mm_Vertical, F.Cu at (163.2, 21.3)
- added J2: Output, Connector_JST:JST_EH_B2B-EH-A_1x02_P2.50mm_Vertical, F.Cu at (114.0, 22.3)
- added J2: Output, Connector_JST:JST_EH_B2B-EH-A_1x02_P2.50mm_Vertical, F.Cu at (57.4, 87.0)
- added J2: Output, Connector_JST:JST_EH_B2B-EH-A_1x02_P2.50mm_Vertical, F.Cu at (81.1, 86.6)
- added J2: Output, Connector_JST:JST_EH_B2B-EH-A_1x02_P2.50mm_Vertical, F.Cu at (31.9, 87.6)
- added J2: Output, Connector_JST:JST_EH_B2B-EH-A_1x02_P2.50mm_Vertical, F.Cu at (57.9, 65.0)
- added J2: Output, Connector_JST:JST_EH_B2B-EH-A_1x02_P2.50mm_Vertical, F.Cu at (81.6, 64.5)
- added J2: Output, Connector_JST:JST_EH_B2B-EH-A_1x02_P2.50mm_Vertical, F.Cu at (195.3, 84.5)
- added J2: Output, Connector_JST:JST_EH_B2B-EH-A_1x02_P2.50mm_Vertical, F.Cu at (32.4, 65.5)
- added J2: Output, Connector_JST:JST_EH_B2B-EH-A_1x02_P2.50mm_Vertical, F.Cu at (59.2, 43.6)
- added J2: Output, Connector_JST:JST_EH_B2B-EH-A_1x02_P2.50mm_Vertical, F.Cu at (82.9, 43.2)
- added J2: Output, Connector_JST:JST_EH_B2B-EH-A_1x02_P2.50mm_Vertical, F.Cu at (33.7, 44.1)
- added J2: Output, Connector_JST:JST_EH_B2B-EH-A_1x02_P2.50mm_Vertical, F.Cu at (219.7, 63.4)
- added J2: Output, Connector_JST:JST_EH_B2B-EH-A_1x02_P2.50mm_Vertical, F.Cu at (243.4, 63.0)
- added J2: Output, Connector_JST:JST_EH_B2B-EH-A_1x02_P2.50mm_Vertical, F.Cu at (194.2, 64.0)
- added J2: Output, Connector_JST:JST_EH_B2B-EH-A_1x02_P2.50mm_Vertical, F.Cu at (219.7, 41.8)
- added J2: Output, Connector_JST:JST_EH_B2B-EH-A_1x02_P2.50mm_Vertical, F.Cu at (243.4, 41.4)
- added J2: Output, Connector_JST:JST_EH_B2B-EH-A_1x02_P2.50mm_Vertical, F.Cu at (194.2, 42.4)
- added LED1: LED, LED_THT:LED_D5.0mm_IRBlack, F.Cu at (237.1, 82.1)
- added LED1: LED, LED_THT:LED_D5.0mm_IRBlack, F.Cu at (236.0, 17.1)
- added LED1: LED, LED_THT:LED_D5.0mm_IRBlack, F.Cu at (212.3, 17.5)
- added LED1: LED, LED_THT:LED_D5.0mm_IRBlack, F.Cu at (186.8, 18.1)
- added LED1: LED, LED_THT:LED_D5.0mm_IRBlack, F.Cu at (153.0, 83.1)
- added LED1: LED, LED_THT:LED_D5.0mm_IRBlack, F.Cu at (129.2, 83.6)
- added LED1: LED, LED_THT:LED_D5.0mm_IRBlack, F.Cu at (103.8, 84.1)
- added LED1: LED, LED_THT:LED_D5.0mm_IRBlack, F.Cu at (154.8, 62.3)
- added LED1: LED, LED_THT:LED_D5.0mm_IRBlack, F.Cu at (131.0, 62.7)
- added LED1: LED, LED_THT:LED_D5.0mm_IRBlack, F.Cu at (105.6, 63.3)
- added LED1: LED, LED_THT:LED_D5.0mm_IRBlack, F.Cu at (154.5, 40.2)
- added LED1: LED, LED_THT:LED_D5.0mm_IRBlack, F.Cu at (213.3, 82.6)
- added LED1: LED, LED_THT:LED_D5.0mm_IRBlack, F.Cu at (130.8, 40.6)
- added LED1: LED, LED_THT:LED_D5.0mm_IRBlack, F.Cu at (105.3, 41.2)
- added LED1: LED, LED_THT:LED_D5.0mm_IRBlack, F.Cu at (155.8, 19.9)
- added LED1: LED, LED_THT:LED_D5.0mm_IRBlack, F.Cu at (132.0, 20.3)
- added LED1: LED, LED_THT:LED_D5.0mm_IRBlack, F.Cu at (106.6, 20.9)
- added LED1: LED, LED_THT:LED_D5.0mm_IRBlack, F.Cu at (73.7, 85.2)
- added LED1: LED, LED_THT:LED_D5.0mm_IRBlack, F.Cu at (50.0, 85.6)
- added LED1: LED, LED_THT:LED_D5.0mm_IRBlack, F.Cu at (24.5, 86.1)
- added LED1: LED, LED_THT:LED_D5.0mm_IRBlack, F.Cu at (74.2, 63.1)
- added LED1: LED, LED_THT:LED_D5.0mm_IRBlack, F.Cu at (50.5, 63.5)
- added LED1: LED, LED_THT:LED_D5.0mm_IRBlack, F.Cu at (187.9, 83.1)
- added LED1: LED, LED_THT:LED_D5.0mm_IRBlack, F.Cu at (25.0, 64.0)
- added LED1: LED, LED_THT:LED_D5.0mm_IRBlack, F.Cu at (75.5, 41.7)
- added LED1: LED, LED_THT:LED_D5.0mm_IRBlack, F.Cu at (51.8, 42.2)
- added LED1: LED, LED_THT:LED_D5.0mm_IRBlack, F.Cu at (26.3, 42.7)
- added LED1: LED, LED_THT:LED_D5.0mm_IRBlack, F.Cu at (236.0, 61.5)
- added LED1: LED, LED_THT:LED_D5.0mm_IRBlack, F.Cu at (212.3, 62.0)
- added LED1: LED, LED_THT:LED_D5.0mm_IRBlack, F.Cu at (186.8, 62.5)
- added LED1: LED, LED_THT:LED_D5.0mm_IRBlack, F.Cu at (236.0, 39.9)
- added LED1: LED, LED_THT:LED_D5.0mm_IRBlack, F.Cu at (212.3, 40.4)
- added LED1: LED, LED_THT:LED_D5.0mm_IRBlack, F.Cu at (186.8, 40.9)
- added R1: 1k, Resistor_THT:R_Axial_DIN0309_L9.0mm_D3.2mm_P12.70mm_Horizontal, F.Cu at (208.6, 88.8)
- added R1: 1k, Resistor_THT:R_Axial_DIN0309_L9.0mm_D3.2mm_P12.70mm_Horizontal, F.Cu at (207.6, 23.8)
- added R1: 1k, Resistor_THT:R_Axial_DIN0309_L9.0mm_D3.2mm_P12.70mm_Horizontal, F.Cu at (231.3, 23.4)
- added R1: 1k, Resistor_THT:R_Axial_DIN0309_L9.0mm_D3.2mm_P12.70mm_Horizontal, F.Cu at (182.1, 24.3)
- added R1: 1k, Resistor_THT:R_Axial_DIN0309_L9.0mm_D3.2mm_P12.70mm_Horizontal, F.Cu at (124.6, 89.8)
- added R1: 1k, Resistor_THT:R_Axial_DIN0309_L9.0mm_D3.2mm_P12.70mm_Horizontal, F.Cu at (148.3, 89.4)
- added R1: 1k, Resistor_THT:R_Axial_DIN0309_L9.0mm_D3.2mm_P12.70mm_Horizontal, F.Cu at (99.1, 90.4)
- added R1: 1k, Resistor_THT:R_Axial_DIN0309_L9.0mm_D3.2mm_P12.70mm_Horizontal, F.Cu at (126.3, 69.0)
- added R1: 1k, Resistor_THT:R_Axial_DIN0309_L9.0mm_D3.2mm_P12.70mm_Horizontal, F.Cu at (150.1, 68.6)
- added R1: 1k, Resistor_THT:R_Axial_DIN0309_L9.0mm_D3.2mm_P12.70mm_Horizontal, F.Cu at (100.9, 69.5)
- added R1: 1k, Resistor_THT:R_Axial_DIN0309_L9.0mm_D3.2mm_P12.70mm_Horizontal, F.Cu at (126.1, 46.9)
- added R1: 1k, Resistor_THT:R_Axial_DIN0309_L9.0mm_D3.2mm_P12.70mm_Horizontal, F.Cu at (232.4, 88.4)
- added R1: 1k, Resistor_THT:R_Axial_DIN0309_L9.0mm_D3.2mm_P12.70mm_Horizontal, F.Cu at (149.8, 46.5)
- added R1: 1k, Resistor_THT:R_Axial_DIN0309_L9.0mm_D3.2mm_P12.70mm_Horizontal, F.Cu at (100.6, 47.5)
- added R1: 1k, Resistor_THT:R_Axial_DIN0309_L9.0mm_D3.2mm_P12.70mm_Horizontal, F.Cu at (127.4, 26.6)
- added R1: 1k, Resistor_THT:R_Axial_DIN0309_L9.0mm_D3.2mm_P12.70mm_Horizontal, F.Cu at (151.1, 26.1)
- added R1: 1k, Resistor_THT:R_Axial_DIN0309_L9.0mm_D3.2mm_P12.70mm_Horizontal, F.Cu at (101.9, 27.1)
- added R1: 1k, Resistor_THT:R_Axial_DIN0309_L9.0mm_D3.2mm_P12.70mm_Horizontal, F.Cu at (45.3, 91.9)
- added R1: 1k, Resistor_THT:R_Axial_DIN0309_L9.0mm_D3.2mm_P12.70mm_Horizontal, F.Cu at (69.0, 91.4)
- added R1: 1k, Resistor_THT:R_Axial_DIN0309_L9.0mm_D3.2mm_P12.70mm_Horizontal, F.Cu at (19.8, 92.4)
- added R1: 1k, Resistor_THT:R_Axial_DIN0309_L9.0mm_D3.2mm_P12.70mm_Horizontal, F.Cu at (45.8, 69.8)
- added R1: 1k, Resistor_THT:R_Axial_DIN0309_L9.0mm_D3.2mm_P12.70mm_Horizontal, F.Cu at (69.5, 69.3)
- added R1: 1k, Resistor_THT:R_Axial_DIN0309_L9.0mm_D3.2mm_P12.70mm_Horizontal, F.Cu at (183.2, 89.4)
- added R1: 1k, Resistor_THT:R_Axial_DIN0309_L9.0mm_D3.2mm_P12.70mm_Horizontal, F.Cu at (20.4, 70.3)
- added R1: 1k, Resistor_THT:R_Axial_DIN0309_L9.0mm_D3.2mm_P12.70mm_Horizontal, F.Cu at (47.1, 48.4)
- added R1: 1k, Resistor_THT:R_Axial_DIN0309_L9.0mm_D3.2mm_P12.70mm_Horizontal, F.Cu at (70.8, 48.0)
- added R1: 1k, Resistor_THT:R_Axial_DIN0309_L9.0mm_D3.2mm_P12.70mm_Horizontal, F.Cu at (21.6, 49.0)
- added R1: 1k, Resistor_THT:R_Axial_DIN0309_L9.0mm_D3.2mm_P12.70mm_Horizontal, F.Cu at (207.6, 68.3)
- added R1: 1k, Resistor_THT:R_Axial_DIN0309_L9.0mm_D3.2mm_P12.70mm_Horizontal, F.Cu at (231.3, 67.8)
- added R1: 1k, Resistor_THT:R_Axial_DIN0309_L9.0mm_D3.2mm_P12.70mm_Horizontal, F.Cu at (182.1, 68.8)
- added R1: 1k, Resistor_THT:R_Axial_DIN0309_L9.0mm_D3.2mm_P12.70mm_Horizontal, F.Cu at (207.6, 46.7)
- added R1: 1k, Resistor_THT:R_Axial_DIN0309_L9.0mm_D3.2mm_P12.70mm_Horizontal, F.Cu at (231.3, 46.2)
- added R1: 1k, Resistor_THT:R_Axial_DIN0309_L9.0mm_D3.2mm_P12.70mm_Horizontal, F.Cu at (182.1, 47.2)
Routing:
- net (no net): track 122.1 -> 2136.5 mm
