File: Diseños pcb/Proyecto semaforo/receptor/receptor.kicad_pcb (KiCad board)
At the start: 2 copper layers, 168 parts, among them J1 Conn_01x03_Male, Q1 2N3904, Q2 2N3904

Commit message: Diseños PCB actualizados
Parts:
- removed the D1 at (266.4, 93.2)
- removed the D1 at (272.5, 19.5)
- removed the D1 at (186.8, 19.5)
- removed the D1 at (229.5, 18.7)
- removed the D1 at (130.2, 93.7)
- removed the D1 at (44.6, 93.7)
- removed the D1 at (87.2, 92.8)
- removed the D1 at (134.1, 67.0)
- removed the D1 at (48.4, 67.0)
- removed the D1 at (91.1, 66.2)
- removed the D1 at (135.6, 42.9)
- removed the D1 at (180.7, 93.2)
- removed the D1 at (49.9, 42.9)
- removed the D1 at (92.6, 42.0)
- removed the D1 at (137.6, 19.8)
- removed the D1 at (94.6, 18.9)
- removed the D1 at (51.9, 19.8)
- removed the D1 at (223.4, 92.3)
- removed the D1 at (268.9, 68.5)
- removed the D1 at (183.2, 68.6)
- removed the D1 at (225.9, 67.7)
- removed the D1 at (271.2, 43.1)
- removed the D1 at (185.5, 43.2)
- removed the D1 at (228.2, 42.3)
- removed the J1 at (190.6, 99.2)
- removed the J1 at (196.7, 25.5)
- removed the J1 at (154.0, 26.4)
- removed the J1 at (239.7, 26.4)
- removed the J1 at (54.5, 99.7)
- removed the J1 at (11.8, 100.6)
- removed the J1 at (97.5, 100.5)
- removed the J1 at (58.3, 73.0)
- removed the J1 at (15.6, 73.9)
- removed the J1 at (101.3, 73.9)
- removed the J1 at (59.8, 48.9)
- removed the J1 at (147.9, 100.1)
- removed the J1 at (17.1, 49.8)
- removed the J1 at (102.8, 49.7)
- removed the J1 at (104.8, 26.6)
- removed the J1 at (61.9, 25.8)
- removed the J1 at (19.2, 26.7)
- removed the J1 at (233.6, 100.0)
- removed the J1 at (193.2, 74.6)
- removed the J1 at (150.5, 75.4)
- removed the J1 at (236.2, 75.4)
- removed the J1 at (195.5, 49.2)
- removed the J1 at (152.8, 50.0)
- removed the J1 at (238.5, 50.0)
- removed the Q1 at (245.0, 95.8)
- removed the Q1 at (251.1, 22.1)
- removed the Q1 at (208.1, 21.3)
- removed the Q1 at (165.4, 22.2)
- removed the Q1 at (108.9, 96.3)
- removed the Q1 at (65.9, 95.5)
- removed the Q1 at (23.2, 96.4)
- removed the Q1 at (112.7, 69.6)
- removed the Q1 at (69.7, 68.8)
- removed the Q1 at (27.0, 69.7)
- removed the Q1 at (114.2, 45.5)
- removed the Q1 at (202.0, 95.0)
- removed the Q1 at (71.2, 44.7)
- removed the Q1 at (28.5, 45.6)
- removed the Q1 at (116.2, 22.4)
- removed the Q1 at (73.2, 21.6)
- removed the Q1 at (30.6, 22.4)
- removed the Q1 at (159.3, 95.9)
- removed the Q1 at (247.6, 71.2)
- removed the Q1 at (204.6, 70.3)
- removed the Q1 at (161.9, 71.2)
- removed the Q1 at (249.9, 45.8)
- removed the Q1 at (206.9, 44.9)
- removed the Q1 at (164.2, 45.8)
- removed the Q2 at (209.3, 94.9)
- removed the Q2 at (215.4, 21.3)
- removed the Q2 at (258.4, 22.1)
- removed the Q2 at (172.7, 22.1)
- removed the Q2 at (73.1, 95.4)
- removed the Q2 at (116.1, 96.2)
- removed the Q2 at (30.5, 96.3)
- removed the Q2 at (76.9, 68.8)
- removed the Q2 at (119.9, 69.6)
- removed the Q2 at (34.3, 69.6)
- removed the Q2 at (78.5, 44.6)
- removed the Q2 at (252.3, 95.7)
- removed the Q2 at (121.5, 45.4)
- removed the Q2 at (35.8, 45.5)
- removed the Q2 at (123.5, 22.3)
- removed the Q2 at (80.5, 21.5)
- removed the Q2 at (37.8, 22.4)
- removed the Q2 at (166.6, 95.8)
- removed the Q2 at (211.8, 70.3)
- removed the Q2 at (254.8, 71.1)
- removed the Q2 at (169.1, 71.1)
- removed the Q2 at (214.1, 44.9)
- removed the Q2 at (257.1, 45.7)
- removed the Q2 at (171.4, 45.7)
- removed the R1 at (156.7, 100.4)
- removed the R1 at (162.8, 26.8)
- removed the R1 at (205.4, 25.9)
- removed the R1 at (248.4, 26.7)
- removed the R1 at (20.5, 100.9)
- removed the R1 at (63.2, 100.1)
- removed the R1 at (106.2, 100.9)
- removed the R1 at (24.3, 74.3)
- removed the R1 at (67.0, 73.4)
- removed the R1 at (110.0, 74.2)
- removed the R1 at (25.8, 50.1)
- removed the R1 at (199.3, 99.5)
- removed the R1 at (68.5, 49.3)
- removed the R1 at (111.5, 50.1)
- removed the R1 at (113.6, 27.0)
- removed the R1 at (70.6, 26.1)
- removed the R1 at (27.9, 27.0)
- removed the R1 at (242.3, 100.4)
- removed the R1 at (159.2, 75.8)
- removed the R1 at (201.9, 74.9)
- removed the R1 at (244.9, 75.7)
- removed the R1 at (161.5, 50.4)
- removed the R1 at (204.2, 49.5)
- removed the R1 at (247.2, 50.3)
- removed the R2 at (260.0, 101.0)
- removed the R2 at (266.1, 27.3)
- removed the R2 at (223.1, 26.5)
- removed the R2 at (180.4, 27.4)
- removed the R2 at (123.8, 101.5)
- removed the R2 at (80.8, 100.7)
- removed the R2 at (38.1, 101.5)
- removed the R2 at (127.6, 74.8)
- removed the R2 at (84.6, 74.0)
- removed the R2 at (41.9, 74.9)
- removed the R2 at (129.1, 50.7)
- removed the R2 at (217.0, 100.1)
- removed the R2 at (86.1, 49.9)
- removed the R2 at (43.5, 50.7)
- removed the R2 at (131.2, 27.6)
- removed the R2 at (88.2, 26.7)
- removed the R2 at (45.5, 27.6)
- removed the R2 at (174.3, 101.0)
- removed the R2 at (262.5, 76.3)
- removed the R2 at (219.5, 75.5)
- removed the R2 at (176.8, 76.4)
- removed the R2 at (264.8, 50.9)
- removed the R2 at (221.8, 50.1)
- removed the R2 at (179.1, 51.0)
- removed the R3 at (241.7, 89.1)
- removed the R3 at (247.8, 15.4)
- removed the R3 at (162.1, 15.5)
- removed the R3 at (204.8, 14.6)
- removed the R3 at (105.6, 89.6)
- removed the R3 at (19.9, 89.6)
- removed the R3 at (62.6, 88.8)
- removed the R3 at (109.4, 62.9)
- removed the R3 at (23.7, 63.0)
- removed the R3 at (66.4, 62.1)
- removed the R3 at (110.9, 38.8)
- removed the R3 at (156.0, 89.1)
- removed the R3 at (25.2, 38.8)
- removed the R3 at (67.9, 38.0)
- removed the R3 at (112.9, 15.7)
- removed the R3 at (69.9, 14.9)
- removed the R3 at (27.2, 15.7)
- removed the R3 at (198.7, 88.3)
- removed the R3 at (244.2, 64.4)
- removed the R3 at (158.6, 64.5)
- removed the R3 at (201.2, 63.6)
- removed the R3 at (246.5, 39.0)
- removed the R3 at (160.9, 39.1)
- removed the R3 at (203.5, 38.2)
- added D1: LED, LED_THT:LED_D5.0mm, F.Cu at (133.3, 148.1)
- added D1: LED, LED_THT:LED_D5.0mm, F.Cu at (70.4, 74.9)
- added D1: LED, LED_THT:LED_D5.0mm, F.Cu at (255.5, 73.7)
- added D1: LED, LED_THT:LED_D5.0mm, F.Cu at (193.8, 74.9)
- added D1: LED, LED_THT:LED_D5.0mm, F.Cu at (254.0, 35.6)
- added D1: LED, LED_THT:LED_D5.0mm, F.Cu at (192.3, 36.8)
- added D1: LED, LED_THT:LED_D5.0mm, F.Cu at (132.3, 36.3)
- added D1: LED, LED_THT:LED_D5.0mm, F.Cu at (68.8, 36.8)
- added D1: LED, LED_THT:LED_D5.0mm, F.Cu at (69.8, 148.6)
- added D1: LED, LED_THT:LED_D5.0mm, F.Cu at (255.0, 147.3)
- added D1: LED, LED_THT:LED_D5.0mm, F.Cu at (193.3, 148.6)
- added D1: LED, LED_THT:LED_D5.0mm, F.Cu at (132.3, 109.2)
- added D1: LED, LED_THT:LED_D5.0mm, F.Cu at (68.8, 109.7)
- added D1: LED, LED_THT:LED_D5.0mm, F.Cu at (254.0, 108.5)
- added D1: LED, LED_THT:LED_D5.0mm, F.Cu at (192.3, 109.7)
- added D1: LED, LED_THT:LED_D5.0mm, F.Cu at (133.9, 74.4)
- added J1: Conn_01x03_Male, Connector_JST:JST_EH_B3B-EH-A_1x03_P2.50mm_Vertical, F.Cu at (93.5, 150.9)
- added J1: Conn_01x03_Male, Connector_JST:JST_EH_B3B-EH-A_1x03_P2.50mm_Vertical, F.Cu at (30.5, 77.7)
- added J1: Conn_01x03_Male, Connector_JST:JST_EH_B3B-EH-A_1x03_P2.50mm_Vertical, F.Cu at (215.6, 76.5)
- added J1: Conn_01x03_Male, Connector_JST:JST_EH_B3B-EH-A_1x03_P2.50mm_Vertical, F.Cu at (153.9, 77.7)
- added J1: Conn_01x03_Male, Connector_JST:JST_EH_B3B-EH-A_1x03_P2.50mm_Vertical, F.Cu at (214.1, 38.4)
- added J1: Conn_01x03_Male, Connector_JST:JST_EH_B3B-EH-A_1x03_P2.50mm_Vertical, F.Cu at (152.4, 39.6)
- added J1: Conn_01x03_Male, Connector_JST:JST_EH_B3B-EH-A_1x03_P2.50mm_Vertical, F.Cu at (92.5, 39.1)
- added J1: Conn_01x03_Male, Connector_JST:JST_EH_B3B-EH-A_1x03_P2.50mm_Vertical, F.Cu at (29.0, 39.6)
- added J1: Conn_01x03_Male, Connector_JST:JST_EH_B3B-EH-A_1x03_P2.50mm_Vertical, F.Cu at (30.0, 151.4)
- added J1: Conn_01x03_Male, Connector_JST:JST_EH_B3B-EH-A_1x03_P2.50mm_Vertical, F.Cu at (215.1, 150.1)
- added J1: Conn_01x03_Male, Connector_JST:JST_EH_B3B-EH-A_1x03_P2.50mm_Vertical, F.Cu at (153.4, 151.4)
- added J1: Conn_01x03_Male, Connector_JST:JST_EH_B3B-EH-A_1x03_P2.50mm_Vertical, F.Cu at (92.5, 112.0)
- added J1: Conn_01x03_Male, Connector_JST:JST_EH_B3B-EH-A_1x03_P2.50mm_Vertical, F.Cu at (29.0, 112.5)
- added J1: Conn_01x03_Male, Connector_JST:JST_EH_B3B-EH-A_1x03_P2.50mm_Vertical, F.Cu at (214.1, 111.3)
- added J1: Conn_01x03_Male, Connector_JST:JST_EH_B3B-EH-A_1x03_P2.50mm_Vertical, F.Cu at (152.4, 112.5)
- added J1: Conn_01x03_Male, Connector_JST:JST_EH_B3B-EH-A_1x03_P2.50mm_Vertical, F.Cu at (94.0, 77.2)
- added Q1: 2N3904, Package_TO_SOT_THT:TO-92_Inline, F.Cu at (39.4, 141.5)
- added Q1: 2N3904, Package_TO_SOT_THT:TO-92_Inline, F.Cu at (225.0, 66.5)
- added Q1: 2N3904, Package_TO_SOT_THT:TO-92_Inline, F.Cu at (163.3, 67.8)
- added Q1: 2N3904, Package_TO_SOT_THT:TO-92_Inline, F.Cu at (103.4, 67.3)
- added Q1: 2N3904, Package_TO_SOT_THT:TO-92_Inline, F.Cu at (223.5, 28.4)
- added Q1: 2N3904, Package_TO_SOT_THT:TO-92_Inline, F.Cu at (161.8, 29.7)
- added Q1: 2N3904, Package_TO_SOT_THT:TO-92_Inline, F.Cu at (101.9, 29.2)
- added Q1: 2N3904, Package_TO_SOT_THT:TO-92_Inline, F.Cu at (38.4, 29.7)
- added Q1: 2N3904, Package_TO_SOT_THT:TO-92_Inline, F.Cu at (224.5, 140.2)
- added Q1: 2N3904, Package_TO_SOT_THT:TO-92_Inline, F.Cu at (162.8, 141.5)
- added Q1: 2N3904, Package_TO_SOT_THT:TO-92_Inline, F.Cu at (102.9, 141.0)
- added Q1: 2N3904, Package_TO_SOT_THT:TO-92_Inline, F.Cu at (38.4, 102.6)
- added Q1: 2N3904, Package_TO_SOT_THT:TO-92_Inline, F.Cu at (223.5, 101.3)
- added Q1: 2N3904, Package_TO_SOT_THT:TO-92_Inline, F.Cu at (161.8, 102.6)
- added Q1: 2N3904, Package_TO_SOT_THT:TO-92_Inline, F.Cu at (101.9, 102.1)
- added Q1: 2N3904, Package_TO_SOT_THT:TO-92_Inline, F.Cu at (39.9, 67.8)
- added Q2: 2N3904, Package_TO_SOT_THT:TO-92_Inline, F.Cu at (113.3, 140.7)
- added Q2: 2N3904, Package_TO_SOT_THT:TO-92_Inline, F.Cu at (50.3, 67.6)
- added Q2: 2N3904, Package_TO_SOT_THT:TO-92_Inline, F.Cu at (235.5, 66.3)
- added Q2: 2N3904, Package_TO_SOT_THT:TO-92_Inline, F.Cu at (173.7, 67.6)
- added Q2: 2N3904, Package_TO_SOT_THT:TO-92_Inline, F.Cu at (233.9, 28.2)
- added Q2: 2N3904, Package_TO_SOT_THT:TO-92_Inline, F.Cu at (172.2, 29.5)
- added Q2: 2N3904, Package_TO_SOT_THT:TO-92_Inline, F.Cu at (112.3, 29.0)
- added Q2: 2N3904, Package_TO_SOT_THT:TO-92_Inline, F.Cu at (48.8, 29.5)
- added Q2: 2N3904, Package_TO_SOT_THT:TO-92_Inline, F.Cu at (49.8, 141.2)
- added Q2: 2N3904, Package_TO_SOT_THT:TO-92_Inline, F.Cu at (234.9, 140.0)
- added Q2: 2N3904, Package_TO_SOT_THT:TO-92_Inline, F.Cu at (173.2, 141.2)
- added Q2: 2N3904, Package_TO_SOT_THT:TO-92_Inline, F.Cu at (112.3, 101.9)
- added Q2: 2N3904, Package_TO_SOT_THT:TO-92_Inline, F.Cu at (48.8, 102.4)
- added Q2: 2N3904, Package_TO_SOT_THT:TO-92_Inline, F.Cu at (233.9, 101.1)
- added Q2: 2N3904, Package_TO_SOT_THT:TO-92_Inline, F.Cu at (172.2, 102.4)
- added Q2: 2N3904, Package_TO_SOT_THT:TO-92_Inline, F.Cu at (113.8, 67.1)
- added R1: 220, Resistor_THT:R_Axial_DIN0309_L9.0mm_D3.2mm_P12.70mm_Horizontal, F.Cu at (102.1, 156.2)
- added R1: 220, Resistor_THT:R_Axial_DIN0309_L9.0mm_D3.2mm_P12.70mm_Horizontal, F.Cu at (224.3, 81.8)
- added R1: 220, Resistor_THT:R_Axial_DIN0309_L9.0mm_D3.2mm_P12.70mm_Horizontal, F.Cu at (39.1, 83.1)
- added R1: 220, Resistor_THT:R_Axial_DIN0309_L9.0mm_D3.2mm_P12.70mm_Horizontal, F.Cu at (162.6, 83.1)
- added R1: 220, Resistor_THT:R_Axial_DIN0309_L9.0mm_D3.2mm_P12.70mm_Horizontal, F.Cu at (222.8, 43.7)
- added R1: 220, Resistor_THT:R_Axial_DIN0309_L9.0mm_D3.2mm_P12.70mm_Horizontal, F.Cu at (161.0, 45.0)
- added R1: 220, Resistor_THT:R_Axial_DIN0309_L9.0mm_D3.2mm_P12.70mm_Horizontal, F.Cu at (101.1, 44.5)
- added R1: 220, Resistor_THT:R_Axial_DIN0309_L9.0mm_D3.2mm_P12.70mm_Horizontal, F.Cu at (37.6, 45.0)
- added R1: 220, Resistor_THT:R_Axial_DIN0309_L9.0mm_D3.2mm_P12.70mm_Horizontal, F.Cu at (223.8, 155.4)
- added R1: 220, Resistor_THT:R_Axial_DIN0309_L9.0mm_D3.2mm_P12.70mm_Horizontal, F.Cu at (38.6, 156.7)
- added R1: 220, Resistor_THT:R_Axial_DIN0309_L9.0mm_D3.2mm_P12.70mm_Horizontal, F.Cu at (162.1, 156.7)
- added R1: 220, Resistor_THT:R_Axial_DIN0309_L9.0mm_D3.2mm_P12.70mm_Horizontal, F.Cu at (101.1, 117.3)
- added R1: 220, Resistor_THT:R_Axial_DIN0309_L9.0mm_D3.2mm_P12.70mm_Horizontal, F.Cu at (222.8, 116.6)
- added R1: 220, Resistor_THT:R_Axial_DIN0309_L9.0mm_D3.2mm_P12.70mm_Horizontal, F.Cu at (37.6, 117.9)
- added R1: 220, Resistor_THT:R_Axial_DIN0309_L9.0mm_D3.2mm_P12.70mm_Horizontal, F.Cu at (161.0, 117.9)
- added R1: 220, Resistor_THT:R_Axial_DIN0309_L9.0mm_D3.2mm_P12.70mm_Horizontal, F.Cu at (102.6, 82.5)
- added R2: 1k, Resistor_THT:R_Axial_DIN0309_L9.0mm_D3.2mm_P12.70mm_Horizontal, F.Cu at (123.4, 142.2)
- added R2: 1k, Resistor_THT:R_Axial_DIN0309_L9.0mm_D3.2mm_P12.70mm_Horizontal, F.Cu at (60.5, 69.1)
- added R2: 1k, Resistor_THT:R_Axial_DIN0309_L9.0mm_D3.2mm_P12.70mm_Horizontal, F.Cu at (245.6, 67.8)
- added R2: 1k, Resistor_THT:R_Axial_DIN0309_L9.0mm_D3.2mm_P12.70mm_Horizontal, F.Cu at (183.9, 69.1)
- added R2: 1k, Resistor_THT:R_Axial_DIN0309_L9.0mm_D3.2mm_P12.70mm_Horizontal, F.Cu at (244.1, 29.7)
- added R2: 1k, Resistor_THT:R_Axial_DIN0309_L9.0mm_D3.2mm_P12.70mm_Horizontal, F.Cu at (182.4, 31.0)
- added R2: 1k, Resistor_THT:R_Axial_DIN0309_L9.0mm_D3.2mm_P12.70mm_Horizontal, F.Cu at (122.4, 30.5)
- added R2: 1k, Resistor_THT:R_Axial_DIN0309_L9.0mm_D3.2mm_P12.70mm_Horizontal, F.Cu at (58.9, 31.0)
- added R2: 1k, Resistor_THT:R_Axial_DIN0309_L9.0mm_D3.2mm_P12.70mm_Horizontal, F.Cu at (59.9, 142.7)
- added R2: 1k, Resistor_THT:R_Axial_DIN0309_L9.0mm_D3.2mm_P12.70mm_Horizontal, F.Cu at (245.1, 141.5)
- added R2: 1k, Resistor_THT:R_Axial_DIN0309_L9.0mm_D3.2mm_P12.70mm_Horizontal, F.Cu at (183.4, 142.7)
- added R2: 1k, Resistor_THT:R_Axial_DIN0309_L9.0mm_D3.2mm_P12.70mm_Horizontal, F.Cu at (122.4, 103.4)
- added R2: 1k, Resistor_THT:R_Axial_DIN0309_L9.0mm_D3.2mm_P12.70mm_Horizontal, F.Cu at (58.9, 103.9)
- added R2: 1k, Resistor_THT:R_Axial_DIN0309_L9.0mm_D3.2mm_P12.70mm_Horizontal, F.Cu at (244.1, 102.6)
- added R2: 1k, Resistor_THT:R_Axial_DIN0309_L9.0mm_D3.2mm_P12.70mm_Horizontal, F.Cu at (182.4, 103.9)
- added R2: 1k, Resistor_THT:R_Axial_DIN0309_L9.0mm_D3.2mm_P12.70mm_Horizontal, F.Cu at (124.0, 68.6)
- added R3: 220, Resistor_THT:R_Axial_DIN0411_L9.9mm_D3.6mm_P12.70mm_Horizontal, F.Cu at (102.4, 148.1)
- added R3: 220, Resistor_THT:R_Axial_DIN0411_L9.9mm_D3.6mm_P12.70mm_Horizontal, F.Cu at (224.5, 73.7)
- added R3: 220, Resistor_THT:R_Axial_DIN0411_L9.9mm_D3.6mm_P12.70mm_Horizontal, F.Cu at (162.8, 74.9)
- added R3: 220, Resistor_THT:R_Axial_DIN0411_L9.9mm_D3.6mm_P12.70mm_Horizontal, F.Cu at (39.4, 74.9)
- added R3: 220, Resistor_THT:R_Axial_DIN0411_L9.9mm_D3.6mm_P12.70mm_Horizontal, F.Cu at (223.0, 35.6)
- added R3: 220, Resistor_THT:R_Axial_DIN0411_L9.9mm_D3.6mm_P12.70mm_Horizontal, F.Cu at (161.3, 36.8)
- added R3: 220, Resistor_THT:R_Axial_DIN0411_L9.9mm_D3.6mm_P12.70mm_Horizontal, F.Cu at (101.3, 36.3)
- added R3: 220, Resistor_THT:R_Axial_DIN0411_L9.9mm_D3.6mm_P12.70mm_Horizontal, F.Cu at (37.8, 36.8)
- added R3: 220, Resistor_THT:R_Axial_DIN0411_L9.9mm_D3.6mm_P12.70mm_Horizontal, F.Cu at (224.0, 147.3)
- added R3: 220, Resistor_THT:R_Axial_DIN0411_L9.9mm_D3.6mm_P12.70mm_Horizontal, F.Cu at (162.3, 148.6)
- added R3: 220, Resistor_THT:R_Axial_DIN0411_L9.9mm_D3.6mm_P12.70mm_Horizontal, F.Cu at (38.9, 148.6)
- added R3: 220, Resistor_THT:R_Axial_DIN0411_L9.9mm_D3.6mm_P12.70mm_Horizontal, F.Cu at (101.3, 109.2)
- added R3: 220, Resistor_THT:R_Axial_DIN0411_L9.9mm_D3.6mm_P12.70mm_Horizontal, F.Cu at (223.0, 108.5)
- added R3: 220, Resistor_THT:R_Axial_DIN0411_L9.9mm_D3.6mm_P12.70mm_Horizontal, F.Cu at (161.3, 109.7)
- added R3: 220, Resistor_THT:R_Axial_DIN0411_L9.9mm_D3.6mm_P12.70mm_Horizontal, F.Cu at (37.8, 109.7)
- added R3: 220, Resistor_THT:R_Axial_DIN0411_L9.9mm_D3.6mm_P12.70mm_Horizontal, F.Cu at (102.9, 74.4)
Routing:
- net (no net): track 4054.5 -> 4256.6 mm
- net Net-(Q1-Pad3): track 0.00 -> 67.7 mm
- net Net-(Q1-Pad1): track 19.9 -> 0.00 mm
- net Net-(D1-Pad2): track 13.3 -> 32.8 mm
- net Net-(J1-Pad3): track 21.6 -> 37.4 mm
- net Net-(J1-Pad1): track 69.3 -> 84.7 mm
- net Net-(J1-Pad2): track 27.2 -> 39.2 mm
- net Net-(D1-Pad1): track 25.0 -> 21.9 mm
